Commit message: Proyecto: cinemática inversa con clicked_point y fix js_current

File: Proyecto/robot_ws/src/robot_description/urdf/robot_rrr.urdf (robot description, URDF)
Before this commit: robot robot, 4 links, 3 joints
Links:
- added link end_effector, mass 0.1; visual sphere radius=0.02
- added link eslabon_fijo, mass 1.5; collision box size=0.04 0.04 0.30; visual box size=0.04 0.04 0.30
- added link world
- link arm_link: mass None -> 1.0; geometry collision box size=0.03 0.03 0.35; visual box size=0.03 0.03 0.35
- link base_link: mass None -> 2.0; geometry collision cylinder length=0.05 radius=0.15; visual cylinder length=0.05 radius=0.15
- link forearm_link: mass None -> 0.8; geometry collision box size=0.025 0.025 0.30; visual box size=0.025 0.025 0.30
- link shoulder_link: mass None -> 1.0; geometry collision cylinder length=0.03 radius=0.12; visual cylinder length=0.03 radius=0.12
Joints:
- added joint joint_ee: type fixed, parent forearm_link, child end_effector, origin xyz=0 0 0.30 rpy=0 0 0
- added joint joint_fijo: type fixed, parent shoulder_link, child eslabon_fijo, origin xyz=0 0 0.03 rpy=0 0 0
- added joint world_to_base: type fixed, parent world, child base_link, origin xyz=0 0 0 rpy=0 0 0
- joint arm_joint: axis 0 0 1 -> 0 1 0; limit lower=-3.14 upper=3.14 effort=10.0 velocity=10.0 -> lower=-1.5708 upper=1.5708 effort=30 velocity=1.0; origin xyz=0.3 0 0 rpy=0 0 0 -> xyz=0 0 0.30 rpy=0 0 0; parent shoulder_link -> eslabon_fijo
- joint forearm_joint: axis 0 0 1 -> 0 1 0; limit lower=-3.14 upper=3.14 effort=10.0 velocity=10.0 -> lower=-1.5708 upper=1.5708 effort=20 velocity=1.0; origin xyz=0.3 0 0 -> xyz=0 0 0.35 rpy=0 0 0
- joint shoulder_joint: limit lower=-3.14 upper=3.14 effort=10.0 velocity=10.0 -> lower=-3.14159 upper=3.14159 effort=50 velocity=1.0; origin xyz=0 0 0 rpy=1.57 0 0 -> xyz=0 0 0.05 rpy=0 0 0
